Commit message: BABY STEPS: IK walk gait...

File: urdf/a1_unitree.urdf (robot description, URDF)
Before this commit: robot a1, 23 links, 22 joints
Links:
- added link cam_L, mass 0.0; collision box size=0.0 0.0 0.0; visual box size=0.04 0.02 0.02
- added link cam_R, mass 0.0; collision box size=0.0 0.0 0.0; visual box size=0.04 0.02 0.02
Joints:
- added joint cam_L_joint: type fixed, parent trunk, child cam_L, origin xyz=0.28 0.05 0.05 rpy=0.0 0.2 0.0, axis 0.0 0.0 0.0, limit lower=0.0 upper=0.0 effort=0.0 velocity=0.0
- added joint cam_R_joint: type fixed, parent trunk, child cam_R, origin xyz=0.28 -0.05 0.05 rpy=0.0 0.2 0.0, axis 0.0 0.0 0.0, limit lower=0.0 upper=0.0 effort=0.0 velocity=0.0

Commit message: IK module added with Docs in Documents folder. Each leg has its own IK params

File: urdf/a1_unitree.urdf (robot description, URDF)
Before this commit: robot a1, 25 links, 24 joints
Links:
- link trunk: mass 6.0 -> 15.0
